Commit message: Spawn 8 thrusters with reading Yaml file

File: surface/rov_simulation/rov_gazebo/worlds/thruster.xacro (robot description, xacro)
@@ -1,16 +1,31 @@
 <?xml version="1.0"?>
 <robot xmlns:xacro="http://www.ros.org/wiki/xacro" name="thruster">
-  <xacro:include filename="inertial_macros.xacro"/>
-  <xacro:macro name="thruster">
+  <xacro:arg name="params_path" default=""/>
+  <!-- Need argument to get from launch file -->
+  <xacro:property name="params_path" value="$(arg params_path)"/>
+  <!-- Need seperate property for xacro inorder processing -->
+  <xacro:property name="params" value="${load_yaml(params_path)}"/>
+  <!-- Read in the yaml dict as mp (short for model parameters) -->
+  <xacro:property name="rov_description" value="${params['rov_description']}"/>
+  <xacro:property name="motor_properties" value="${rov_description['motor']}"/>
+  <xacro:macro name="thruster" params="name motor reflectx reflecty">
+    <xacro:property name="thruster_name" value="thruster_${motor}_${name}"/>
+    <xacro:property name="motor_object" value="${motor_properties[motor]}"/>
+    <xacro:property name="width_from_center" value="${motor_object['width_from_center']}"/>
+    <xacro:property name="length_from_center" value="${motor_object['length_from_center']}"/>
+    <xacro:property name="height_from_center" value="${motor_object['height_from_center']}"/>
+    <xacro:property name="roll" value="${motor_object['roll']}"/>
+    <xacro:property name="pitch" value="${motor_object['pitch']}"/>
+    <xacro:property name="yaw" value="${motor_object['yaw']}"/>
     <origin rpy="3.141592 0 0" xyz="0 0 0"/>
-    <joint name="body_thruster_joint" type="fixed">
+    <joint name="body_${thruster_name}_joint" type="fixed">
       <parent link="body"/>
-      <child link="thruster_body"/>
-      <origin rpy="0 0 0" xyz="0 0 0.5"/>
+      <child link="${thruster_name}_body"/>
+      <origin xyz="${width_from_center*reflectx} ${length_from_center*reflecty} ${height_from_center}" rpy= "${roll} ${pitch} ${reflecty*reflectx*yaw }"/>
     </joint>
-    <link name='thruster_body'>
+    <link name='${thruster_name}_body'>
       <origin rpy="0 0 0" xyz="0 0 0"/>
       <xacro:inertial_cylinder mass="0.5" length="0.05" radius="0.01">
-        <origin rpy="0 0 0" xyz="0 0 0"/>
+      <origin rpy="0 0 0" xyz="0 0 0"/>
       </xacro:inertial_cylinder>
       <visual>
@@ -25,12 +40,12 @@
       </collision>
     </link>
-    <link name='thruster_blade'>
+    <link name='${thruster_name}_blade'>
       <origin rpy="0 0 0" xyz="0 0 0"/>
       <inertial>
-        <mass value="1.5"/>
+        <mass value="0.5"/>
         <inertia ixx="0.4" ixy="0" ixz="0" iyy="0.4" iyz="0" izz="0.8"/>
       </inertial>
       <visual>
-        <origin rpy="-0.7853981633974483 0 0" xyz="0.3 0 0"/>
+        <origin rpy="-0.7853981633974483 0 0" xyz="0.03 0 0"/>
         <geometry>
           <box size="0.04 0.02 0.005"/>
@@ -38,5 +53,5 @@
       </visual>
       <collision>
-        <origin rpy="-0.7853981633974483 0 0" xyz="0.3 0 0"/>
+        <origin rpy="-0.7853981633974483 0 0" xyz="0.03 0 0"/>
         <geometry>
           <box size="0.04 0.02 0.005"/>
@@ -44,5 +59,5 @@
       </collision>
       <visual>
-        <origin rpy="-0.7853981633974483 0 1.5707963267948966" xyz="0 0.3 0"/>
+        <origin rpy="-0.7853981633974483 0 1.5707963267948966" xyz="0 0.03 0"/>
         <geometry>
           <box size="0.04 0.02 0.005"/>
@@ -50,5 +65,5 @@
       </visual>
       <collision>
-        <origin rpy="-0.7853981633974483 0 1.5707963267948966" xyz="0 0.3 0"/>
+        <origin rpy="-0.7853981633974483 0 1.5707963267948966" xyz="0 0.03 0"/>
         <geometry>
           <box size="0.04 0.02 0.005"/>
@@ -56,5 +71,5 @@
       </collision>
       <visual>
-        <origin rpy="0.7853981633974483 0 0" xyz="-0.3 0 0"/>
+        <origin rpy="0.7853981633974483 0 0" xyz="-0.03 0 0"/>
         <geometry>
           <box size="0.04 0.02 0.005"/>
@@ -62,5 +77,5 @@
       </visual>
       <collision>
-        <origin rpy="0.7853981633974483 0 0" xyz="-0.3 0 0"/>
+        <origin rpy="0.7853981633974483 0 0" xyz="-0.03 0 0"/>
         <geometry>
           <box size="0.04 0.02 0.005"/>
@@ -68,5 +83,5 @@
       </collision>
       <visual>
-        <origin rpy="0.7853981633974483 0 1.5707963267948966" xyz="0 -0.3 0"/>
+        <origin rpy="0.7853981633974483 0 1.5707963267948966" xyz="0 -0.03 0"/>
         <geometry>
           <box size="0.04 0.02 0.005"/>
@@ -74,5 +89,5 @@
       </visual>
       <collision>
-        <origin rpy="0.7853981633974483 0 1.5707963267948966" xyz="0 -0.3 0"/>
+        <origin rpy="0.7853981633974483 0 1.5707963267948966" xyz="0 -0.03 0"/>
         <geometry>
           <box size="0.04 0.02 0.005"/>
@@ -80,7 +95,7 @@
       </collision>
     </link>
-    <joint name='thruster_body_blade_joint' type='revolute'>
-      <parent link="thruster_body"/>
-      <child link="thruster_blade"/>
+    <joint name='${thruster_name}_body_blade_joint' type='revolute'>
+      <parent link="${thruster_name}_body"/>
+      <child link="${thruster_name}_blade"/>
       <axis xyz="0 0 1"/>
       <limit lower="-1e+12" upper="1e+12" effort="-1" velocity="-1"/>
@@ -100,5 +115,5 @@
         <upward>0 -0.707106781186547 -0.707106781186547</upward>
         <forward>0 -0.707106781186547 0.707106781186547</forward>
-        <link_name>thruster_blade</link_name>
+        <link_name>${thruster_name}_blade</link_name>
         <cp>0.35 0 0</cp>
       </plugin>
@@ -116,5 +131,5 @@
         <upward>-0.707106781186547 0 -0.707106781186547</upward>
         <forward>-0.707106781186547 0 0.707106781186547</forward>
-        <link_name>thruster_blade</link_name>
+        <link_name>${thruster_name}_blade</link_name>
         <cp>0 -0.35 0</cp>
       </plugin>
@@ -132,5 +147,5 @@
         <upward>0 0.707106781186547 -0.707106781186547</upward>
         <forward>0 -0.707106781186547 -0.707106781186547</forward>
-        <link_name>thruster_blade</link_name>
+        <link_name>${thruster_name}_blade</link_name>
         <cp>-0.35 0 0</cp>
       </plugin>
@@ -148,5 +163,5 @@
         <upward>0.707106781186547 0 -0.707106781186547</upward>
         <forward>0.707106781186547 0 0.707106781186547</forward>
-        <link_name>thruster_blade</link_name>
+        <link_name>${thruster_name}_blade</link_name>
         <cp>0 0.35 0</cp>
       </plugin>
@@ -154,8 +169,15 @@
         filename="ignition-gazebo-apply-joint-force-system"
         name="ignition::gazebo::systems::ApplyJointForce">
-        <joint_name>thruster_body_blade_joint</joint_name>
+        <joint_name>${thruster_name}_body_blade_joint</joint_name>
       </plugin>
     </gazebo>
   </xacro:macro>
-  <xacro:thruster/>
+  <xacro:thruster name="front_left" motor="top" reflectx="1" reflecty="1"/>
+  <xacro:thruster name="front_right" motor="top" reflectx="1" reflecty="-1"/>
+  <xacro:thruster name="back_left" motor="top" reflectx="-1" reflecty="1"/>
+  <xacro:thruster name="back_right" motor="top" reflectx="-1" reflecty="-1"/>
+  <xacro:thruster name="front_left" motor="bottom" reflectx="1" reflecty="1"/>
+  <xacro:thruster name="front_right" motor="bottom" reflectx="1" reflecty="-1"/>
+  <xacro:thruster name="back_left" motor="bottom" reflectx="-1" reflecty="1"/>
+  <xacro:thruster name="back_right" motor="bottom" reflectx="-1" reflecty="-1"/>
 </robot>

Commit message: Add ArduPilot plugin

File: surface/rov_simulation/rov_gazebo/worlds/thruster.xacro (robot description, xacro)
@@ -181,3 +181,38 @@
   <xacro:thruster name="back_left" motor="bottom" reflectx="-1" reflecty="1"/>
   <xacro:thruster name="back_right" motor="bottom" reflectx="-1" reflecty="-1"/>
+  <gazebo>
+    <plugin name="ArduPilotPlugin" filename="libArduPilotPlugin.so">
+      <!-- Port settings -->
+      <fdm_addr>127.0.0.1</fdm_addr>
+      <fdm_port_in>9002</fdm_port_in>
+      <connectionTimeoutMaxCount>5</connectionTimeoutMaxCount>
+      <lock_step>1</lock_step>
+      <!-- Transform from the Ignition Gazebo body frame (x-forward, y-left, z-up)
+          to the ArduPilot body frame (x-forward, y-right, z-down) -->
+      <modelXYZToAirplaneXForwardZDown>0 0 0 3.141592653589793 0 0</modelXYZToAirplaneXForwardZDown>
+      <!-- Transform from the Ignition Gazebo world frame (ENU)
+          to the ArduPilot world frame (NED) -->
+      <gazeboXYZToNED>0 0 0 3.141592653589793 0 1.5707963267948966</gazeboXYZToNED>
+      <xacro:macro name="thruster_control" params="channel jointName">
+        <!-- Thrusters -->
+        <control channel="${channel}">
+          <jointName>${jointName}</jointName>
+          <servo_min>1100</servo_min>
+          <servo_max>1900</servo_max>
+          <type>COMMAND</type>
+          <cmd_topic>/model/rov/joint/${jointName}_joint/cmd_force</cmd_topic>
+          <offset>-0.5</offset>
+          <multiplier>100</multiplier>
+        </control>
+      </xacro:macro>
+      <xacro:thruster_control channel="0" jointName="thruster_top_front_left_body_blade_joint"/>
+      <xacro:thruster_control channel="1" jointName="thruster_top_front_right_body_blade_joint"/>
+      <xacro:thruster_control channel="2" jointName="thruster_top_back_left_body_blade_joint"/>
+      <xacro:thruster_control channel="3" jointName="thruster_top_back_right_body_blade_joint"/>
+      <xacro:thruster_control channel="4" jointName="thruster_bottom_front_left_body_blade_joint"/>
+      <xacro:thruster_control channel="5" jointName="thruster_bottom_front_right_body_blade_joint"/>
+      <xacro:thruster_control channel="6" jointName="thruster_bottom_back_left_body_blade_joint"/>
+      <xacro:thruster_control channel="7" jointName="thruster_bottom_back_right_body_blade_joint"/>
+    </plugin>
+  </gazebo>
 </robot>
