Commit message: neutrally bouyant

File: surface/rov_simulation/rov_description/urdf/rov.xacro (robot description, xacro)
@@ -16,8 +16,7 @@
       <xacro:property name="motor_height" value="${motor_properties['dimension']['height']}"/>
         <link name="base_link">
-            <gravity>0</gravity>
             <!-- no basis-->
             <inertial>
-                <mass value="1"/>
+                <mass value="136.382"/>
                 <inertia ixx="1e-3" ixy="0" ixz="0" iyy="1e-3" iyz="0" izz="1e-3" />
             </inertial>
@@ -37,5 +36,4 @@
                 </geometry>
                 <!-- no basis-->
-                <contact_coefficients mu="0" kp="1000.0" kd="1.0"/>
             </collision>
         </link>

Commit message: deleted plugins

File: surface/rov_simulation/rov_description/urdf/rov.xacro (robot description, xacro)
@@ -109,114 +109,3 @@
       </gazebo>
       -->
-      <!-- From BlueROV2 example -->
-      <!-- Hydrodynamics plugin -->
-        <plugin filename="ignition-gazebo-hydrodynamics-system"
-        name="ignition::gazebo::systems::Hydrodynamics"><link_name>base_link</link_name>
-          <water_density>1000</water_density>
-          <!-- Added mass: -->
-          <xDotU>0</xDotU>
-          <yDotV>0</yDotV>`
-          <zDotW>0</zDotW>
-          <kDotP>0</kDotP>
-          <mDotQ>0</mDotQ>
-          <nDotR>0</nDotR>
-          <!-- First order stability derivative: -->
-          <xU>0</xU>
-          <yV>0</yV>
-          <zW>0</zW>
-          <kP>0</kP>
-          <mQ>0</mQ>
-          <nR>0</nR>
-          <!-- Second order stability derivative: -->
-          <xUU>-33.800000000000004</xUU>
-          <yVV>-54.26875</yVV>
-          <zWW>-73.37135</zWW>
-          <kPP>-4.0</kPP>
-          <mQQ>-4.0</mQQ>
-          <nRR>-4.0</nRR>
-        </plugin>
-        <xacro:macro name="thruster" params="name motor reflectx reflecty">
-          <xacro:property name="thruster_name" value="thruster_${motor}_${name}"/>
-          <xacro:property name="motor_object" value="${motor_properties[motor]}"/>
-          <xacro:property name="width_from_center" value="${motor_object['width_from_center']}"/>
-          <xacro:property name="length_from_center" value="${motor_object['length_from_center']}"/>
-          <xacro:property name="height_from_center" value="${motor_object['height_from_center']}"/>
-          <xacro:property name="roll" value="${motor_object['roll']}"/>
-          <xacro:property name="pitch" value="${motor_object['pitch']}"/>
-          <xacro:property name="yaw" value="${motor_object['yaw']}"/>
-          <joint name="${thruster_name}_joint" type="fixed">
-            <parent link = "base_link"/>
-            <child link= "${thruster_name}_link"/>
-            <origin xyz="${width_from_center*reflectx} ${length_from_center*reflecty} ${height_from_center}" rpy= "${roll} ${pitch} ${reflecty*reflectx*yaw }"/>
-          </joint>
-          <link name="${thruster_name}_link">
-            <collision>
-              <geometry>
-                <cylinder radius="${motor_radius}" length="${motor_height}"/>
-              </geometry>
-            </collision>
-            <visual>
-              <geometry>
-                <cylinder radius="${motor_radius}" length="${motor_height}"/>
-              </geometry>
-            </visual>
-            <!-- small vals-->
-            <inertial>
-              <mass value="1e-5" />
-              <inertia ixx="1e-6" ixy="0" ixz="0" iyy="1e-6" iyz="0" izz="1e-6" />
-            </inertial>
-          </link>
-          <plugin filename="ignition-gazebo-thruster-system"
-        name="ignition::gazebo::systems::Thruster">>
-            <namespace>rov</namespace>
-            <joint_name>"${thruster_name}_joint"</joint_name>
-            <thrust_coefficient>0.02</thrust_coefficient>
-            <fluid_density>1000</fluid_density>
-            <propeller_diameter>${motor_radius*2}</propeller_diameter>
-            <velocity_control>true</velocity_control>
-            <use_angvel_cmd>False</use_angvel_cmd>
-          </plugin>
-        </xacro:macro>
-    <!-- TODO: FOR LOOPS MAYBE?-->
-      <xacro:thruster name="front_left" motor="top" reflectx="1" reflecty="1"/>
-      <xacro:thruster name="front_right" motor="top" reflectx="1" reflecty="-1"/>
-      <xacro:thruster name="back_left" motor="top" reflectx="-1" reflecty="1"/>
-      <xacro:thruster name="back_right" motor="top" reflectx="-1" reflecty="-1"/>
-      <xacro:thruster name="front_left" motor="bottom" reflectx="1" reflecty="1"/>
-      <xacro:thruster name="front_right" motor="bottom" reflectx="1" reflecty="-1"/>
-      <xacro:thruster name="back_left" motor="bottom" reflectx="-1" reflecty="1"/>
-      <xacro:thruster name="back_right" motor="bottom" reflectx="-1" reflecty="-1"/>
-      <plugin name="ArduPilotPlugin" filename="libArduPilotPlugin.so">
-          <!-- Port settings -->
-          <fdm_addr>127.0.0.1</fdm_addr>
-          <fdm_port_in>9002</fdm_port_in>
-          <connectionTimeoutMaxCount>5</connectionTimeoutMaxCount>
-          <lock_step>1</lock_step>
-          <!-- Transform from the Ignition Gazebo body frame (x-forward, y-left, z-up)
-              to the ArduPilot body frame (x-forward, y-right, z-down) -->
-          <modelXYZToAirplaneXForwardZDown>0 0 0 3.141592653589793 0 0</modelXYZToAirplaneXForwardZDown>
-          <!-- Transform from the Ignition Gazebo world frame (ENU)
-              to the ArduPilot world frame (NED) -->
-          <gazeboXYZToNED>0 0 0 3.141592653589793 0 1.5707963267948966</gazeboXYZToNED>
-          <xacro:macro name="thruster_control" params="channel jointName">
-            <!-- Thrusters -->
-            <control channel="${channel}">
-              <jointName>${jointName}_joint</jointName>
-              <servo_min>1100</servo_min>
-              <servo_max>1900</servo_max>
-              <type>COMMAND</type>
-              <cmd_topic>/model/rov/joint/${jointName}_joint/cmd_thrust</cmd_topic>
-              <offset>-0.5</offset>
-              <multiplier>100</multiplier>
-            </control>
-          </xacro:macro>
-          <xacro:thruster_control channel="0" jointName="top_front_left"/>
-          <xacro:thruster_control channel="1" jointName="top_front_right"/>
-          <xacro:thruster_control channel="2" jointName="top_back_left"/>
-          <xacro:thruster_control channel="3" jointName="top_back_right"/>
-          <xacro:thruster_control channel="4" jointName="bottom_front_left"/>
-          <xacro:thruster_control channel="5" jointName="bottom_front_right"/>
-          <xacro:thruster_control channel="6" jointName="bottom_back_left"/>
-          <xacro:thruster_control channel="7" jointName="bottom_back_right"/>
-        </plugin>
 </robot>
