Commit message: Add thruster blade direction

File: surface/rov_gazebo/description/thruster.xacro (robot description, xacro)
@@ -9,5 +9,5 @@
   <xacro:property name="rov_description" value="${params['rov_description']}"/>
   <xacro:property name="motor_properties" value="${rov_description['motor']}"/>
-  <xacro:macro name="thruster" params="name motor reflectx reflecty">
+  <xacro:macro name="thruster" params="name motor reflectx reflecty reflect_blade">
     <xacro:property name="thruster_name" value="thruster_${motor}_${name}"/>
     <xacro:property name="motor_object" value="${motor_properties[motor]}"/>
@@ -43,51 +43,51 @@
       <origin rpy="0 0 0" xyz="0 0 0"/>
       <inertial>
-        <mass value="0.5"/>
+        <mass value="0.46"/>
         <inertia ixx="0.4" ixy="0" ixz="0" iyy="0.4" iyz="0" izz="0.8"/>
       </inertial>
       <visual>
-        <origin rpy="-0.7853981633974483 0 0" xyz="0.03 0 0"/>
-        <geometry>
-          <box size="0.04 0.02 0.005"/>
-        </geometry>
-      </visual>
-      <collision>
-        <origin rpy="-0.7853981633974483 0 0" xyz="0.03 0 0"/>
-        <geometry>
-          <box size="0.04 0.02 0.005"/>
-        </geometry>
-      </collision>
-      <visual>
-        <origin rpy="-0.7853981633974483 0 1.5707963267948966" xyz="0 0.03 0"/>
-        <geometry>
-          <box size="0.04 0.02 0.005"/>
-        </geometry>
-      </visual>
-      <collision>
-        <origin rpy="-0.7853981633974483 0 1.5707963267948966" xyz="0 0.03 0"/>
-        <geometry>
-          <box size="0.04 0.02 0.005"/>
-        </geometry>
-      </collision>
-      <visual>
-        <origin rpy="0.7853981633974483 0 0" xyz="-0.03 0 0"/>
-        <geometry>
-          <box size="0.04 0.02 0.005"/>
-        </geometry>
-      </visual>
-      <collision>
-        <origin rpy="0.7853981633974483 0 0" xyz="-0.03 0 0"/>
-        <geometry>
-          <box size="0.04 0.02 0.005"/>
-        </geometry>
-      </collision>
-      <visual>
-        <origin rpy="0.7853981633974483 0 1.5707963267948966" xyz="0 -0.03 0"/>
-        <geometry>
-          <box size="0.04 0.02 0.005"/>
-        </geometry>
-      </visual>
-      <collision>
-        <origin rpy="0.7853981633974483 0 1.5707963267948966" xyz="0 -0.03 0"/>
+        <origin rpy="${-0.7853981633974483 * reflect_blade} 0 0" xyz="0.03 0 0"/>
+        <geometry>
+          <box size="0.04 0.02 0.005"/>
+        </geometry>
+      </visual>
+      <collision>
+        <origin rpy="${-0.7853981633974483 * reflect_blade} 0 0" xyz="0.03 0 0"/>
+        <geometry>
+          <box size="0.04 0.02 0.005"/>
+        </geometry>
+      </collision>
+      <visual>
+        <origin rpy="${-0.7853981633974483 * reflect_blade} 0 1.5707963267948966" xyz="0 0.03 0"/>
+        <geometry>
+          <box size="0.04 0.02 0.005"/>
+        </geometry>
+      </visual>
+      <collision>
+        <origin rpy="${-0.7853981633974483 * reflect_blade} 0 1.5707963267948966" xyz="0 0.03 0"/>
+        <geometry>
+          <box size="0.04 0.02 0.005"/>
+        </geometry>
+      </collision>
+      <visual>
+        <origin rpy="${0.7853981633974483 * reflect_blade} 0 0" xyz="-0.03 0 0"/>
+        <geometry>
+          <box size="0.04 0.02 0.005"/>
+        </geometry>
+      </visual>
+      <collision>
+        <origin rpy="${0.7853981633974483 * reflect_blade} 0 0" xyz="-0.03 0 0"/>
+        <geometry>
+          <box size="0.04 0.02 0.005"/>
+        </geometry>
+      </collision>
+      <visual>
+        <origin rpy="${0.7853981633974483 * reflect_blade} 0 1.5707963267948966" xyz="0 -0.03 0"/>
+        <geometry>
+          <box size="0.04 0.02 0.005"/>
+        </geometry>
+      </visual>
+      <collision>
+        <origin rpy="${0.7853981633974483 * reflect_blade} 0 1.5707963267948966" xyz="0 -0.03 0"/>
         <geometry>
           <box size="0.04 0.02 0.005"/>
@@ -173,12 +173,12 @@
     </gazebo>
   </xacro:macro>
-  <xacro:thruster name="front_left" motor="top" reflectx="1" reflecty="1"/>
-  <xacro:thruster name="front_right" motor="top" reflectx="1" reflecty="-1"/>
-  <xacro:thruster name="back_left" motor="top" reflectx="-1" reflecty="1"/>
-  <xacro:thruster name="back_right" motor="top" reflectx="-1" reflecty="-1"/>
-  <xacro:thruster name="front_left" motor="bottom" reflectx="1" reflecty="1"/>
-  <xacro:thruster name="front_right" motor="bottom" reflectx="1" reflecty="-1"/>
-  <xacro:thruster name="back_left" motor="bottom" reflectx="-1" reflecty="1"/>
-  <xacro:thruster name="back_right" motor="bottom" reflectx="-1" reflecty="-1"/>
+  <xacro:thruster name="front_left" motor="top" reflectx="1" reflecty="1" reflect_blade="-1"/>
+  <xacro:thruster name="front_right" motor="top" reflectx="1" reflecty="-1" reflect_blade="-1"/>
+  <xacro:thruster name="back_left" motor="top" reflectx="-1" reflecty="1" reflect_blade="1"/>
+  <xacro:thruster name="back_right" motor="top" reflectx="-1" reflecty="-1" reflect_blade="1"/>
+  <xacro:thruster name="front_left" motor="bottom" reflectx="1" reflecty="1" reflect_blade="1"/>
+  <xacro:thruster name="front_right" motor="bottom" reflectx="1" reflecty="-1" reflect_blade="-1"/>
+  <xacro:thruster name="back_left" motor="bottom" reflectx="-1" reflecty="1" reflect_blade="-1"/>
+  <xacro:thruster name="back_right" motor="bottom" reflectx="-1" reflecty="-1" reflect_blade="1"/>
   <gazebo>
     <plugin name="ArduPilotPlugin" filename="libArduPilotPlugin.so">

Commit message: Remove ardupilot plugin

File: surface/rov_gazebo/description/thruster.xacro (robot description, xacro)
@@ -121,40 +121,3 @@
   <xacro:thruster name="back_left" motor="bottom" reflectx="-1" reflecty="1" reflect_blade="-1"/>
   <xacro:thruster name="back_right" motor="bottom" reflectx="-1" reflecty="-1" reflect_blade="1"/>
-  <gazebo>
-    <plugin name="ArduPilotPlugin" filename="libArduPilotPlugin.so">
-      <!-- Port settings -->
-      <fdm_addr>127.0.0.1</fdm_addr>
-      <fdm_port_in>9002</fdm_port_in>
-      <fdm_port_out>9003</fdm_port_out>
-      <!-- <imuName>rov::body::imu_sensor</imuName> -->
-      <connectionTimeoutMaxCount>5</connectionTimeoutMaxCount>
-      <lock_step>1</lock_step>
-      <!-- Transform from the Ignition Gazebo body frame (x-forward, y-left, z-up)
-          to the ArduPilot body frame (x-forward, y-right, z-down) -->
-      <modelXYZToAirplaneXForwardZDown>0 0 0 3.141592653589793 0 0</modelXYZToAirplaneXForwardZDown>
-      <!-- Transform from the Ignition Gazebo world frame (ENU)
-          to the ArduPilot world frame (NED) -->
-      <gazeboXYZToNED>0 0 0 3.141592653589793 0 1.5707963267948966</gazeboXYZToNED>
-      <xacro:macro name="thruster_control" params="channel jointName">
-        <!-- Thrusters -->
-        <control channel="${channel}">
-          <jointName>${jointName}</jointName>
-          <servo_min>1100</servo_min>
-          <servo_max>1900</servo_max>
-          <type>COMMAND</type>
-          <cmd_topic>/model/rov/joint/${jointName}_joint/cmd_force</cmd_topic>
-          <offset>-0.5</offset>
-          <multiplier>100</multiplier>
-        </control>
-      </xacro:macro>
-      <xacro:thruster_control channel="0" jointName="thruster_top_front_right_body_blade_joint"/>
-      <xacro:thruster_control channel="1" jointName="thruster_top_front_left_body_blade_joint"/>
-      <xacro:thruster_control channel="2" jointName="thruster_top_back_right_body_blade_joint"/>
-      <xacro:thruster_control channel="3" jointName="thruster_top_back_left_body_blade_joint"/>
-      <xacro:thruster_control channel="4" jointName="thruster_bottom_front_right_body_blade_joint"/>
-      <xacro:thruster_control channel="5" jointName="thruster_bottom_front_left_body_blade_joint"/>
-      <xacro:thruster_control channel="6" jointName="thruster_bottom_back_right_body_blade_joint"/>
-      <xacro:thruster_control channel="7" jointName="thruster_bottom_back_left_body_blade_joint"/>
-    </plugin>
-  </gazebo>
 </robot>

Commit message: Remove thruster blade direction

File: surface/rov_gazebo/description/thruster.xacro (robot description, xacro)
@@ -9,5 +9,5 @@
   <xacro:property name="rov_description" value="${params['rov_description']}"/>
   <xacro:property name="motor_properties" value="${rov_description['motor']}"/>
-  <xacro:macro name="thruster" params="name motor reflectx reflecty reflect_blade">
+  <xacro:macro name="thruster" params="name motor reflectx reflecty">
     <xacro:property name="thruster_name" value="thruster_${motor}_${name}"/>
     <xacro:property name="motor_object" value="${motor_properties[motor]}"/>
@@ -22,5 +22,5 @@
       <parent link="body"/>
       <child link="${thruster_name}_body"/>
-      <origin xyz="${width_from_center*reflectx} ${length_from_center*reflecty} ${height_from_center}" rpy= "${roll} ${pitch} ${reflecty*reflectx*yaw }"/>
+      <origin xyz="${width_from_center*reflectx} ${length_from_center*reflecty} ${height_from_center}" rpy= "${roll} ${pitch} ${reflecty*reflectx*yaw}"/>
     </joint>
     <link name='${thruster_name}_body'>
@@ -47,5 +47,5 @@
       </inertial>
       <visual>
-        <origin rpy="${-0.7853981633974483 * reflect_blade} 0 0" xyz="0.03 0 0"/>
+        <origin rpy="0.7853981633974483 0 0" xyz="0.03 0 0"/>
         <geometry>
           <box size="0.04 0.02 0.005"/>
@@ -53,5 +53,5 @@
       </visual>
       <collision>
-        <origin rpy="${-0.7853981633974483 * reflect_blade} 0 0" xyz="0.03 0 0"/>
+        <origin rpy="0.7853981633974483 0 0" xyz="0.03 0 0"/>
         <geometry>
           <box size="0.04 0.02 0.005"/>
@@ -59,5 +59,5 @@
       </collision>
       <visual>
-        <origin rpy="${-0.7853981633974483 * reflect_blade} 0 1.5707963267948966" xyz="0 0.03 0"/>
+        <origin rpy="0.7853981633974483 0 1.5707963267948966" xyz="0 0.03 0"/>
         <geometry>
           <box size="0.04 0.02 0.005"/>
@@ -65,5 +65,5 @@
       </visual>
       <collision>
-        <origin rpy="${-0.7853981633974483 * reflect_blade} 0 1.5707963267948966" xyz="0 0.03 0"/>
+        <origin rpy="0.7853981633974483 0 1.5707963267948966" xyz="0 0.03 0"/>
         <geometry>
           <box size="0.04 0.02 0.005"/>
@@ -71,5 +71,5 @@
       </collision>
       <visual>
-        <origin rpy="${0.7853981633974483 * reflect_blade} 0 0" xyz="-0.03 0 0"/>
+        <origin rpy="-0.7853981633974483 0 0" xyz="-0.03 0 0"/>
         <geometry>
           <box size="0.04 0.02 0.005"/>
@@ -77,5 +77,5 @@
       </visual>
       <collision>
-        <origin rpy="${0.7853981633974483 * reflect_blade} 0 0" xyz="-0.03 0 0"/>
+        <origin rpy="-0.7853981633974483 0 0" xyz="-0.03 0 0"/>
         <geometry>
           <box size="0.04 0.02 0.005"/>
@@ -83,5 +83,5 @@
       </collision>
       <visual>
-        <origin rpy="${0.7853981633974483 * reflect_blade} 0 1.5707963267948966" xyz="0 -0.03 0"/>
+        <origin rpy="-0.7853981633974483 0 1.5707963267948966" xyz="0 -0.03 0"/>
         <geometry>
           <box size="0.04 0.02 0.005"/>
@@ -89,5 +89,5 @@
       </visual>
       <collision>
-        <origin rpy="${0.7853981633974483 * reflect_blade} 0 1.5707963267948966" xyz="0 -0.03 0"/>
+        <origin rpy="-0.7853981633974483 0 1.5707963267948966" xyz="0 -0.03 0"/>
         <geometry>
           <box size="0.04 0.02 0.005"/>
@@ -107,5 +107,5 @@
           <namespace>rov</namespace>
           <joint_name>${thruster_name}_body_blade_joint</joint_name>
-          <thrust_coefficient>${0.004422 * reflect_blade}</thrust_coefficient>
+          <thrust_coefficient>0.004422</thrust_coefficient>
           <fluid_density>1000</fluid_density>
           <propeller_diameter>0.2</propeller_diameter>
@@ -113,11 +113,11 @@
     </gazebo>
   </xacro:macro>
-  <xacro:thruster name="front_left" motor="top" reflectx="1" reflecty="1" reflect_blade="-1"/>
-  <xacro:thruster name="front_right" motor="top" reflectx="1" reflecty="-1" reflect_blade="-1"/>
-  <xacro:thruster name="back_left" motor="top" reflectx="-1" reflecty="1" reflect_blade="1"/>
-  <xacro:thruster name="back_right" motor="top" reflectx="-1" reflecty="-1" reflect_blade="1"/>
-  <xacro:thruster name="front_left" motor="bottom" reflectx="1" reflecty="1" reflect_blade="1"/>
-  <xacro:thruster name="front_right" motor="bottom" reflectx="1" reflecty="-1" reflect_blade="-1"/>
-  <xacro:thruster name="back_left" motor="bottom" reflectx="-1" reflecty="1" reflect_blade="-1"/>
-  <xacro:thruster name="back_right" motor="bottom" reflectx="-1" reflecty="-1" reflect_blade="1"/>
+  <xacro:thruster name="front_left" motor="top" reflectx="1" reflecty="1"/>
+  <xacro:thruster name="front_right" motor="top" reflectx="1" reflecty="-1"/>
+  <xacro:thruster name="back_left" motor="top" reflectx="-1" reflecty="1"/>
+  <xacro:thruster name="back_right" motor="top" reflectx="-1" reflecty="-1"/>
+  <xacro:thruster name="front_left" motor="bottom" reflectx="1" reflecty="1"/>
+  <xacro:thruster name="front_right" motor="bottom" reflectx="1" reflecty="-1"/>
+  <xacro:thruster name="back_left" motor="bottom" reflectx="-1" reflecty="1"/>
+  <xacro:thruster name="back_right" motor="bottom" reflectx="-1" reflecty="-1"/>
 </robot>

Commit message: Change thruster position

File: surface/rov_gazebo/description/thruster.xacro (robot description, xacro)
@@ -25,5 +25,4 @@
     </joint>
     <link name='${thruster_name}_body'>
-      <origin rpy="0 0 0" xyz="0 0 0"/>
       <xacro:inertial_cylinder mass="0.5" length="0.05" radius="0.01">
       <origin rpy="0 0 0" xyz="0 0 0"/>
