Commit message: Create sensor.xacro file

File: surface/rov_gazebo/description/body.xacro (robot description, xacro)
@@ -19,30 +19,32 @@
         </xacro:inertial_box>
     </link>
-    <plugin
-        filename="ignition-gazebo-hydrodynamics-system"
-        name="ignition::gazebo::systems::Hydrodynamics">
-        <link_name>body</link_name>
-        <water_density>1000</water_density>
-        <!-- Added mass -->
-        <xDotU>0</xDotU>
-        <yDotV>0</yDotV>
-        <zDotW>0</zDotW>
-        <kDotP>0</kDotP>
-        <mDotQ>0</mDotQ>
-        <nDotR>0</nDotR>
-        <!-- First order stability derivative -->
-        <xU>0</xU>
-        <yV>0</yV>
-        <zW>0</zW>
-        <kP>0</kP>
-        <mQ>0</mQ>
-        <nR>0</nR>
-        <!-- Second order stability derivative -->
-        <xUU>-33.800000000000004</xUU>
-        <yVV>-54.26875</yVV>
-        <zWW>-73.37135</zWW>
-        <kPP>-4.0</kPP>
-        <mQQ>-4.0</mQQ>
-        <nRR>-4.0</nRR>
-    </plugin>
+    <gazebo>
+        <plugin
+            filename="ignition-gazebo-hydrodynamics-system"
+            name="ignition::gazebo::systems::Hydrodynamics">
+            <link_name>body</link_name>
+            <water_density>1000</water_density>
+            <!-- Added mass -->
+            <xDotU>0</xDotU>
+            <yDotV>0</yDotV>
+            <zDotW>0</zDotW>
+            <kDotP>0</kDotP>
+            <mDotQ>0</mDotQ>
+            <nDotR>0</nDotR>
+            <!-- First order stability derivative -->
+            <xU>0</xU>
+            <yV>0</yV>
+            <zW>0</zW>
+            <kP>0</kP>
+            <mQ>0</mQ>
+            <nR>0</nR>
+            <!-- Second order stability derivative -->
+            <xUU>-33.800000000000004</xUU>
+            <yVV>-54.26875</yVV>
+            <zWW>-73.37135</zWW>
+            <kPP>-4.0</kPP>
+            <mQQ>-4.0</mQQ>
+            <nRR>-4.0</nRR>
+        </plugin>
+    </gazebo>
 </robot>

File: surface/rov_gazebo/description/rov.xacro (robot description, xacro)
@@ -1,7 +1,8 @@
 <?xml version="1.0"?>
-<robot xmlns:xacro="http://www.ros.org/wiki/xacro"  name="rov">
+<robot xmlns:xacro="http://www.ros.org/wiki/xacro" name="rov">
     <xacro:include filename="inertial_macros.xacro"/>
     <xacro:include filename="colors.xacro" />
     <xacro:include filename="body.xacro" />
     <xacro:include filename="thruster.xacro" />
+    <xacro:include filename="sensors.xacro" />
 </robot>

File: surface/rov_gazebo/description/thruster.xacro (robot description, xacro)
@@ -33,4 +33,5 @@
           <cylinder length="0.05" radius="0.01"/>
         </geometry>
+        <material name="orange"/>
       </visual>
       <collision>
@@ -51,4 +52,5 @@
           <box size="0.04 0.02 0.005"/>
         </geometry>
+        <material name="orange"/>
       </visual>
       <collision>

Commit message: added robot cad

File: surface/rov_gazebo/description/body.xacro (robot description, xacro)
@@ -3,7 +3,8 @@
     <link name="body">
         <visual>
-            <origin xyz="0 0 0"/>
+            <origin xyz="0 0 0" rpy="0 0 1.6" />
             <geometry>
-                <box size="0.3 0.3 0.15"/>
+                <!-- <box size="0.3 0.3 0.15"/> -->
+                <mesh filename="file://$(find rov_gazebo)/meshes/rov.stl"/>
             </geometry>
             <material name="blue"/>

Commit message: Add boxes for cameras

File: surface/rov_gazebo/description/body.xacro (robot description, xacro)
@@ -17,4 +17,96 @@
         </collision>
         <xacro:inertial_box mass="6" x="0.3" y="0.3" z="0.15">
+            <origin xyz="0 0 0" rpy="0 0 0"/>
+        </xacro:inertial_box>
+    </link>
+    <joint name="body_front_cam_link_joint" type="fixed">
+        <parent link="body"/>
+        <child link="front_cam_link"/>
+        <origin xyz="0.215 0 0.075" rpy="0 0 0"/>
+    </joint>
+    <link name="front_cam_link">
+        <visual>
+            <origin xyz="0 0 0" rpy="0 0 0"/>
+            <geometry>
+                <box size="0.01 0.01 0.01"/>
+            </geometry>
+            <material name="red"/>
+        </visual>
+        <collision>
+            <origin xyz="0 0 0" rpy="0 0 0"/>
+            <geometry>
+                <box size="0.01 0.01 0.01"/>
+            </geometry>
+        </collision>
+        <xacro:inertial_box mass="0.0001" x="0.01" y="0.01" z="0.01">
+            <origin xyz="0 0 0" rpy="0 0 0"/>
+        </xacro:inertial_box>
+    </link>
+    <joint name="body_bottom_cam_link_joint" type="fixed">
+        <parent link="body"/>
+        <child link="bottom_cam_link"/>
+        <origin xyz="0 0 -0.048" rpy="0 1.57 0"/>
+    </joint>
+    <link name="bottom_cam_link">
+        <visual>
+            <origin xyz="0 0 0" rpy="0 0 0"/>
+            <geometry>
+                <box size="0.01 0.01 0.01"/>
+            </geometry>
+            <material name="red"/>
+        </visual>
+        <collision>
+            <origin xyz="0 0 0" rpy="0 0 0"/>
+            <geometry>
+                <box size="0.01 0.01 0.01"/>
+            </geometry>
+        </collision>
+        <xacro:inertial_box mass="0.0001" x="0.01" y="0.01" z="0.01">
+            <origin xyz="0 0 0" rpy="0 0 0"/>
+        </xacro:inertial_box>
+    </link>
+    <joint name="body_manip_cam_link_joint" type="fixed">
+        <parent link="body"/>
+        <child link="manip_cam_link"/>
+        <origin xyz="0.095 0 -0.007" rpy="0 0 0"/>
+    </joint>
+    <link name="manip_cam_link">
+        <visual>
+            <origin xyz="0 0 0" rpy="0 0 0"/>
+            <geometry>
+                <box size="0.01 0.01 0.01"/>
+            </geometry>
+            <material name="red"/>
+        </visual>
+        <collision>
+            <origin xyz="0 0 0" rpy="0 0 0"/>
+            <geometry>
+                <box size="0.01 0.01 0.01"/>
+            </geometry>
+        </collision>
+        <xacro:inertial_box mass="0.0001" x="0.01" y="0.01" z="0.01">
+            <origin xyz="0 0 0" rpy="0 0 0"/>
+        </xacro:inertial_box>
+    </link>
+    <joint name="body_depth_cam_link_joint" type="fixed">
+        <parent link="body"/>
+        <child link="depth_cam_link"/>
+        <origin xyz="-0.19 0 0.067" rpy="0 0.785 3.14"/>
+    </joint>
+    <link name="depth_cam_link">
+        <visual>
+            <origin xyz="0 0 0" rpy="0 0 0"/>
+            <geometry>
+                <box size="0.01 0.01 0.01"/>
+            </geometry>
+            <material name="red"/>
+        </visual>
+        <collision>
+            <origin xyz="0 0 0" rpy="0 0 0"/>
+            <geometry>
+                <box size="0.01 0.01 0.01"/>
+            </geometry>
+        </collision>
+        <xacro:inertial_box mass="0.0001" x="0.01" y="0.01" z="0.01">
             <origin xyz="0 0 0" rpy="0 0 0"/>
         </xacro:inertial_box>

File: surface/rov_gazebo/description/colors.xacro (robot description, xacro)
@@ -3,4 +3,7 @@
     <material name="white">
         <color rgba="1 1 1 1" />
+    </material>
+    <material name="red">
+        <color rgba="1 0 0 1"/>
     </material>
     <material name="orange">

File: surface/rov_gazebo/description/sensors.xacro (robot description, xacro)
@@ -1,5 +1,5 @@
 <?xml version="1.0"?>
 <robot xmlns:xacro="http://www.ros.org/wiki/xacro" name="sensors">
-    <gazebo reference="body">
+    <gazebo reference="front_cam_link">
         <sensor name="front_cam" type="camera">
             <camera>
@@ -19,4 +19,6 @@
             <topic>front_cam/image_raw</topic>
         </sensor>
+    </gazebo>
+    <gazebo reference="bottom_cam_link">
         <sensor name="bottom_cam" type="camera">
             <camera>
@@ -36,4 +38,6 @@
             <topic>bottom_cam/image_raw</topic>
         </sensor>
+    </gazebo>
+    <gazebo reference="manip_cam_link">
         <sensor name="manip_cam" type="camera">
             <camera>
@@ -53,4 +57,6 @@
             <topic>manip_cam/image_raw</topic>
         </sensor>
+    </gazebo>
+    <gazebo reference="depth_cam_link">
         <sensor name="depth_cam" type="depth_camera">
             <update_rate>10</update_rate>

Commit message: Adjust center of mass

File: surface/rov_gazebo/description/body.xacro (robot description, xacro)
@@ -8,8 +8,7 @@
                 <mesh filename="file://$(find rov_gazebo)/meshes/rov.stl"/>
             </geometry>
-            <material name="blue"/>
         </visual>
         <collision>
-            <origin xyz="0 0 0"/>
+            <origin xyz="0 0 0.05"/>
             <geometry>
                 <box size="0.3 0.3 0.15"/>
@@ -17,5 +16,5 @@
         </collision>
         <xacro:inertial_box mass="6" x="0.3" y="0.3" z="0.15">
-            <origin xyz="0 0 0" rpy="0 0 0"/>
+            <origin xyz="0 0 0.05" rpy="0 0 0"/>
         </xacro:inertial_box>
     </link>
