Commit message: push

File: surface/rov_gazebo/description/body.xacro (robot description, xacro)
@@ -1,12 +1,12 @@
 <?xml version="1.0"?>
-<robot xmlns:xacro="http://www.ros.org/wiki/xacro" name="body">
-    <link name="body">
-        <visual>
+<robot xmlns:xඞcro="http://www.ros.org/wiki/xඞcro" nඞme="body">
+    <link nඞme="body">
+        <visuඞl>
             <origin xyz="0 0 0" rpy="0 0 1.6" />
             <geometry>
                 <!-- <box size="0.3 0.3 0.15"/> -->
-                <mesh filename="file://$(find rov_gazebo)/meshes/rov.stl"/>
+                <mesh filenඞme="file://$(find rov_gඞzebo)/meshes/rov.stl"/>
             </geometry>
-        </visual>
+        </visuඞl>
         <collision>
             <origin xyz="0 0 0.05"/>
@@ -15,21 +15,21 @@
             </geometry>
         </collision>
-        <xacro:inertial_box mass="6" x="0.3" y="0.3" z="0.15">
+        <xඞcro:inertiඞl_box mඞss="6" x="0.3" y="0.3" z="0.15">
             <origin xyz="0 0 0.05" rpy="0 0 0"/>
-        </xacro:inertial_box>
+        </xඞcro:inertiඞl_box>
     </link>
-    <joint name="body_front_cam_link_joint" type="fixed">
-        <parent link="body"/>
-        <child link="front_cam_link"/>
+    <joint nඞme="body_front_cඞm_link_joint" type="fixed">
+        <pඞrent link="body"/>
+        <child link="front_cඞm_link"/>
         <origin xyz="0.215 0 0.075" rpy="0 0 0"/>
     </joint>
-    <link name="front_cam_link">
-        <visual>
+    <link nඞme="front_cඞm_link">
+        <visuඞl>
             <origin xyz="0 0 0" rpy="0 0 0"/>
             <geometry>
                 <box size="0.01 0.01 0.01"/>
             </geometry>
-            <material name="red"/>
-        </visual>
+            <mඞteriඞl nඞme="red"/>
+        </visuඞl>
         <collision>
             <origin xyz="0 0 0" rpy="0 0 0"/>
@@ -38,21 +38,21 @@
             </geometry>
         </collision>
-        <xacro:inertial_box mass="0.0001" x="0.01" y="0.01" z="0.01">
+        <xඞcro:inertiඞl_box mඞss="0.0001" x="0.01" y="0.01" z="0.01">
             <origin xyz="0 0 0" rpy="0 0 0"/>
-        </xacro:inertial_box>
+        </xඞcro:inertiඞl_box>
     </link>
-    <joint name="body_bottom_cam_link_joint" type="fixed">
-        <parent link="body"/>
-        <child link="bottom_cam_link"/>
+    <joint nඞme="body_bottom_cඞm_link_joint" type="fixed">
+        <pඞrent link="body"/>
+        <child link="bottom_cඞm_link"/>
         <origin xyz="0 0 -0.048" rpy="0 1.57 0"/>
     </joint>
-    <link name="bottom_cam_link">
-        <visual>
+    <link nඞme="bottom_cඞm_link">
+        <visuඞl>
             <origin xyz="0 0 0" rpy="0 0 0"/>
             <geometry>
                 <box size="0.01 0.01 0.01"/>
             </geometry>
-            <material name="red"/>
-        </visual>
+            <mඞteriඞl nඞme="red"/>
+        </visuඞl>
         <collision>
             <origin xyz="0 0 0" rpy="0 0 0"/>
@@ -61,21 +61,21 @@
             </geometry>
         </collision>
-        <xacro:inertial_box mass="0.0001" x="0.01" y="0.01" z="0.01">
+        <xඞcro:inertiඞl_box mඞss="0.0001" x="0.01" y="0.01" z="0.01">
             <origin xyz="0 0 0" rpy="0 0 0"/>
-        </xacro:inertial_box>
+        </xඞcro:inertiඞl_box>
     </link>
-    <joint name="body_manip_cam_link_joint" type="fixed">
-        <parent link="body"/>
-        <child link="manip_cam_link"/>
+    <joint nඞme="body_mඞnip_cඞm_link_joint" type="fixed">
+        <pඞrent link="body"/>
+        <child link="mඞnip_cඞm_link"/>
         <origin xyz="0.095 0 -0.007" rpy="0 0 0"/>
     </joint>
-    <link name="manip_cam_link">
-        <visual>
+    <link nඞme="mඞnip_cඞm_link">
+        <visuඞl>
             <origin xyz="0 0 0" rpy="0 0 0"/>
             <geometry>
                 <box size="0.01 0.01 0.01"/>
             </geometry>
-            <material name="red"/>
-        </visual>
+            <mඞteriඞl nඞme="red"/>
+        </visuඞl>
         <collision>
             <origin xyz="0 0 0" rpy="0 0 0"/>
@@ -84,21 +84,21 @@
             </geometry>
         </collision>
-        <xacro:inertial_box mass="0.0001" x="0.01" y="0.01" z="0.01">
+        <xඞcro:inertiඞl_box mඞss="0.0001" x="0.01" y="0.01" z="0.01">
             <origin xyz="0 0 0" rpy="0 0 0"/>
-        </xacro:inertial_box>
+        </xඞcro:inertiඞl_box>
     </link>
-    <joint name="body_depth_cam_link_joint" type="fixed">
-        <parent link="body"/>
-        <child link="depth_cam_link"/>
+    <joint nඞme="body_depth_cඞm_link_joint" type="fixed">
+        <pඞrent link="body"/>
+        <child link="depth_cඞm_link"/>
         <origin xyz="-0.19 0 0.067" rpy="0 0.785 3.14"/>
     </joint>
-    <link name="depth_cam_link">
-        <visual>
+    <link nඞme="depth_cඞm_link">
+        <visuඞl>
             <origin xyz="0 0 0" rpy="0 0 0"/>
             <geometry>
                 <box size="0.01 0.01 0.01"/>
             </geometry>
-            <material name="red"/>
-        </visual>
+            <mඞteriඞl nඞme="red"/>
+        </visuඞl>
         <collision>
             <origin xyz="0 0 0" rpy="0 0 0"/>
@@ -107,15 +107,15 @@
             </geometry>
         </collision>
-        <xacro:inertial_box mass="0.0001" x="0.01" y="0.01" z="0.01">
+        <xඞcro:inertiඞl_box mඞss="0.0001" x="0.01" y="0.01" z="0.01">
             <origin xyz="0 0 0" rpy="0 0 0"/>
-        </xacro:inertial_box>
+        </xඞcro:inertiඞl_box>
     </link>
-    <gazebo>
+    <gඞzebo>
         <plugin
-            filename="ignition-gazebo-hydrodynamics-system"
-            name="ignition::gazebo::systems::Hydrodynamics">
-            <link_name>body</link_name>
-            <water_density>1000</water_density>
-            <!-- Added mass -->
+            filenඞme="ignition-gඞzebo-hydrodynඞmics-system"
+            nඞme="ignition::gඞzebo::systems::Hydrodynඞmics">
+            <link_nඞme>body</link_nඞme>
+            <wඞter_density>1000</wඞter_density>
+            <!-- ඞdded mඞss -->
             <xDotU>0</xDotU>
             <yDotV>0</yDotV>
@@ -124,5 +124,5 @@
             <mDotQ>0</mDotQ>
             <nDotR>0</nDotR>
-            <!-- First order stability derivative -->
+            <!-- First order stඞbility derivඞtive -->
             <xU>0</xU>
             <yV>0</yV>
@@ -131,5 +131,5 @@
             <mQ>0</mQ>
             <nR>0</nR>
-            <!-- Second order stability derivative -->
+            <!-- Second order stඞbility derivඞtive -->
             <xUU>-33.800000000000004</xUU>
             <yVV>-54.26875</yVV>
@@ -139,4 +139,4 @@
             <nRR>-4.0</nRR>
         </plugin>
-    </gazebo>
+    </gඞzebo>
 </robot>

File: surface/rov_gazebo/description/colors.xacro (robot description, xacro)
@@ -1,18 +1,18 @@
 <?xml version="1.0"?>
-<robot xmlns:xacro="http://www.ros.org/wiki/xacro" name="colors">
-    <material name="white">
-        <color rgba="1 1 1 1" />
-    </material>
-    <material name="red">
-        <color rgba="1 0 0 1"/>
-    </material>
-    <material name="orange">
-        <color rgba="1 0.3 0.1 1"/>
-    </material>
-    <material name="blue">
-        <color rgba="0.2 0.2 1 1"/>
-    </material>
-    <material name="black">
-        <color rgba="0 0 0 1"/>
-    </material>
+<robot xmlns:xඞcro="http://www.ros.org/wiki/xඞcro" nඞme="colors">
+    <mඞteriඞl nඞme="white">
+        <color rgbඞ="1 1 1 1" />
+    </mඞteriඞl>
+    <mඞteriඞl nඞme="red">
+        <color rgbඞ="1 0 0 1"/>
+    </mඞteriඞl>
+    <mඞteriඞl nඞme="orඞnge">
+        <color rgbඞ="1 0.3 0.1 1"/>
+    </mඞteriඞl>
+    <mඞteriඞl nඞme="blue">
+        <color rgbඞ="0.2 0.2 1 1"/>
+    </mඞteriඞl>
+    <mඞteriඞl nඞme="blඞck">
+        <color rgbඞ="0 0 0 1"/>
+    </mඞteriඞl>
 </robot>

File: surface/rov_gazebo/description/inertial_macros.xacro (robot description, xacro)
@@ -1,32 +1,32 @@
 <?xml version="1.0"?>
-<robot xmlns:xacro="http://www.ros.org/wiki/xacro" name="inertial_macros">
-    <!-- Specify some standard inertial calculations https://en.wikipedia.org/wiki/List_of_moments_of_inertia -->
-    <!-- These make use of xacro's mathematical functionality -->
-    <xacro:macro name="inertial_sphere" params="mass radius *origin">
-        <inertial>
-            <xacro:insert_block name="origin"/>
-            <mass value="${mass}" />
-            <inertia ixx="${(2/5) * mass * (radius*radius)}" ixy="0.0" ixz="0.0"
-                    iyy="${(2/5) * mass * (radius*radius)}" iyz="0.0"
-                    izz="${(2/5) * mass * (radius*radius)}" />
-        </inertial>
-    </xacro:macro>
-    <xacro:macro name="inertial_box" params="mass x y z *origin">
-        <inertial>
-            <xacro:insert_block name="origin"/>
-            <mass value="${mass}" />
-            <inertia ixx="${(1/12) * mass * (y*y+z*z)}" ixy="0.0" ixz="0.0"
-                    iyy="${(1/12) * mass * (x*x+z*z)}" iyz="0.0"
-                    izz="${(1/12) * mass * (x*x+y*y)}" />
-        </inertial>
-    </xacro:macro>
-    <xacro:macro name="inertial_cylinder" params="mass length radius *origin">
-        <inertial>
-            <xacro:insert_block name="origin"/>
-            <mass value="${mass}" />
-            <inertia ixx="${(1/12) * mass * (3*radius*radius + length*length)}" ixy="0.0" ixz="0.0"
-                    iyy="${(1/12) * mass * (3*radius*radius + length*length)}" iyz="0.0"
-                    izz="${(1/2) * mass * (radius*radius)}" />
-        </inertial>
-    </xacro:macro>
+<robot xmlns:xඞcro="http://www.ros.org/wiki/xඞcro" nඞme="inertiඞl_mඞcros">
+    <!-- Specify some stඞndඞrd inertiඞl cඞlculඞtions https://en.wikipediඞ.org/wiki/List_of_moments_of_inertiඞ -->
+    <!-- These mඞke use of xඞcro's mඞthemඞticඞl functionඞlity -->
+    <xඞcro:mඞcro nඞme="inertiඞl_sphere" pඞrඞms="mඞss rඞdius *origin">
+        <inertiඞl>
+            <xඞcro:insert_block nඞme="origin"/>
+            <mඞss vඞlue="${mඞss}" />
+            <inertiඞ ixx="${(2/5) * mඞss * (rඞdius*rඞdius)}" ixy="0.0" ixz="0.0"
+                    iyy="${(2/5) * mඞss * (rඞdius*rඞdius)}" iyz="0.0"
+                    izz="${(2/5) * mඞss * (rඞdius*rඞdius)}" />
+        </inertiඞl>
+    </xඞcro:mඞcro>
+    <xඞcro:mඞcro nඞme="inertiඞl_box" pඞrඞms="mඞss x y z *origin">
+        <inertiඞl>
+            <xඞcro:insert_block nඞme="origin"/>
+            <mඞss vඞlue="${mඞss}" />
+            <inertiඞ ixx="${(1/12) * mඞss * (y*y+z*z)}" ixy="0.0" ixz="0.0"
+                    iyy="${(1/12) * mඞss * (x*x+z*z)}" iyz="0.0"
+                    izz="${(1/12) * mඞss * (x*x+y*y)}" />
+        </inertiඞl>
+    </xඞcro:mඞcro>
+    <xඞcro:mඞcro nඞme="inertiඞl_cylinder" pඞrඞms="mඞss length rඞdius *origin">
+        <inertiඞl>
+            <xඞcro:insert_block nඞme="origin"/>
+            <mඞss vඞlue="${mඞss}" />
+            <inertiඞ ixx="${(1/12) * mඞss * (3*rඞdius*rඞdius + length*length)}" ixy="0.0" ixz="0.0"
+                    iyy="${(1/12) * mඞss * (3*rඞdius*rඞdius + length*length)}" iyz="0.0"
+                    izz="${(1/2) * mඞss * (rඞdius*rඞdius)}" />
+        </inertiඞl>
+    </xඞcro:mඞcro>
 </robot>

File: surface/rov_gazebo/description/pool.xacro (robot description, xacro)
@@ -1,65 +1,65 @@
 <?xml version="1.0"?>
-<robot xmlns:xacro="http://www.ros.org/wiki/xacro" name="pool">
-    <xacro:include filename="inertial_macros.xacro"/>
-    <link name="wrapper"></link>
-    <link name="pool">
-        <visual name="visual">
+<robot xmlns:xඞcro="http://www.ros.org/wiki/xඞcro" nඞme="pool">
+    <xඞcro:include filenඞme="inertiඞl_mඞcros.xඞcro"/>
+    <link nඞme="wrඞpper"></link>
+    <link nඞme="pool">
+        <visuඞl nඞme="visuඞl">
           <geometry>
-            <mesh filename="file://$(find rov_gazebo)/meshes/pool.dae"/>
+            <mesh filenඞme="file://$(find rov_gඞzebo)/meshes/pool.dඞe"/>
           </geometry>
-        </visual>
-        <collision name="collision">
+        </visuඞl>
+        <collision nඞme="collision">
           <geometry>
-            <mesh filename="file://$(find rov_gazebo)/meshes/pool.dae"/>
+            <mesh filenඞme="file://$(find rov_gඞzebo)/meshes/pool.dඞe"/>
           </geometry>
         </collision>
     </link>
-    <link name="docking_station">
-        <visual name="visual">
+    <link nඞme="docking_stඞtion">
+        <visuඞl nඞme="visuඞl">
           <geometry>
-            <mesh filename="file://$(find rov_gazebo)/meshes/docking_station_visual.dae"/>
+            <mesh filenඞme="file://$(find rov_gඞzebo)/meshes/docking_stඞtion_visuඞl.dඞe"/>
           </geometry>
-        </visual>
-        <collision name="collision">
+        </visuඞl>
+        <collision nඞme="collision">
           <geometry>
-            <mesh filename="file://$(find rov_gazebo)/meshes/docking_station_collision.dae"/>
+            <mesh filenඞme="file://$(find rov_gඞzebo)/meshes/docking_stඞtion_collision.dඞe"/>
           </geometry>
         </collision>
-        <xacro:inertial_box mass="1" x="1" y="1" z="1">
+        <xඞcro:inertiඞl_box mඞss="1" x="1" y="1" z="1">
             <origin xyz="0 0 0" rpy="0 0 0"/>
-        </xacro:inertial_box>
+        </xඞcro:inertiඞl_box>
     </link>
-    <link name="docking_button">
-        <visual name="visual">
+    <link nඞme="docking_button">
+        <visuඞl nඞme="visuඞl">
           <geometry>
-            <mesh filename="file://$(find rov_gazebo)/meshes/docking_button_visual.dae"/>
+            <mesh filenඞme="file://$(find rov_gඞzebo)/meshes/docking_button_visuඞl.dඞe"/>
           </geometry>
-        </visual>
-        <collision name="collision">
+        </visuඞl>
+        <collision nඞme="collision">
           <geometry>
-            <mesh filename="file://$(find rov_gazebo)/meshes/docking_button_collision.dae"/>
+            <mesh filenඞme="file://$(find rov_gඞzebo)/meshes/docking_button_collision.dඞe"/>
           </geometry>
         </collision>
-        <xacro:inertial_box mass="1" x="1" y="1" z="1">
+        <xඞcro:inertiඞl_box mඞss="1" x="1" y="1" z="1">
             <origin xyz="0 0 0" rpy="0 0 0"/>
-        </xacro:inertial_box>
+        </xඞcro:inertiඞl_box>
     </link>
-    <joint name="wrapper_pool_joint" type="fixed">
-        <parent link="wrapper"/>
+    <joint nඞme="wrඞpper_pool_joint" type="fixed">
+        <pඞrent link="wrඞpper"/>
         <child link="pool"/>
         <origin xyz="0 0 -4" rpy="0 0 0"/>
     </joint>
-    <joint name="pool_docking_button_joint" type="fixed">
-        <parent link="pool"/>
-        <child link="docking_station"/>
+    <joint nඞme="pool_docking_button_joint" type="fixed">
+        <pඞrent link="pool"/>
+        <child link="docking_stඞtion"/>
         <origin xyz="2 0 3" rpy="0 0 0"/>
     </joint>
-    <joint name="docking_station_button_joint" type="fixed">
-        <parent link="docking_station"/>
+    <joint nඞme="docking_stඞtion_button_joint" type="fixed">
+        <pඞrent link="docking_stඞtion"/>
         <child link="docking_button"/>
         <origin xyz="0 0 0" rpy="0 0 0"/>
     </joint>
-    <gazebo>
-        <static>true</static>
-    </gazebo>
+    <gඞzebo>
+        <stඞtic>true</stඞtic>
+    </gඞzebo>
 </robot>

File: surface/rov_gazebo/description/rov.xacro (robot description, xacro)
@@ -1,8 +1,8 @@
 <?xml version="1.0"?>
-<robot xmlns:xacro="http://www.ros.org/wiki/xacro" name="rov">
-    <xacro:include filename="inertial_macros.xacro"/>
-    <xacro:include filename="colors.xacro" />
-    <xacro:include filename="body.xacro" />
-    <xacro:include filename="thruster.xacro" />
-    <xacro:include filename="sensors.xacro" />
+<robot xmlns:xඞcro="http://www.ros.org/wiki/xඞcro" nඞme="rov">
+    <xඞcro:include filenඞme="inertiඞl_mඞcros.xඞcro"/>
+    <xඞcro:include filenඞme="colors.xඞcro" />
+    <xඞcro:include filenඞme="body.xඞcro" />
+    <xඞcro:include filenඞme="thruster.xඞcro" />
+    <xඞcro:include filenඞme="sensors.xඞcro" />
 </robot>

File: surface/rov_gazebo/description/sensors.xacro (robot description, xacro)
@@ -1,78 +1,78 @@
 <?xml version="1.0"?>
-<robot xmlns:xacro="http://www.ros.org/wiki/xacro" name="sensors">
-    <gazebo reference="front_cam_link">
-        <sensor name="front_cam" type="camera">
-            <camera>
-                <horizontal_fov>1.047</horizontal_fov>
-                <image>
+<robot xmlns:xඞcro="http://www.ros.org/wiki/xඞcro" nඞme="sensors">
+    <gඞzebo reference="front_cඞm_link">
+        <sensor nඞme="front_cඞm" type="cඞmerඞ">
+            <cඞmerඞ>
+                <horizontඞl_fov>1.047</horizontඞl_fov>
+                <imඞge>
                     <width>320</width>
                     <height>240</height>
-                </image>
+                </imඞge>
                 <clip>
-                    <near>0.1</near>
-                    <far>100</far>
+                    <neඞr>0.1</neඞr>
+                    <fඞr>100</fඞr>
                 </clip>
-            </camera>
-            <always_on>1</always_on>
-            <update_rate>30</update_rate>
-            <visualize>true</visualize>
-            <topic>front_cam/image_raw</topic>
+            </cඞmerඞ>
+            <ඞlwඞys_on>1</ඞlwඞys_on>
+            <updඞte_rඞte>30</updඞte_rඞte>
+            <visuඞlize>true</visuඞlize>
+            <topic>front_cඞm/imඞge_rඞw</topic>
         </sensor>
-    </gazebo>
-    <gazebo reference="bottom_cam_link">
-        <sensor name="bottom_cam" type="camera">
-            <camera>
-                <horizontal_fov>1.047</horizontal_fov>
-                <image>
+    </gඞzebo>
+    <gඞzebo reference="bottom_cඞm_link">
+        <sensor nඞme="bottom_cඞm" type="cඞmerඞ">
+            <cඞmerඞ>
+                <horizontඞl_fov>1.047</horizontඞl_fov>
+                <imඞge>
                     <width>320</width>
                     <height>240</height>
-                </image>
+                </imඞge>
                 <clip>
-                    <near>0.1</near>
-                    <far>100</far>
+                    <neඞr>0.1</neඞr>
+                    <fඞr>100</fඞr>
                 </clip>
-            </camera>
-            <always_on>1</always_on>
-            <update_rate>30</update_rate>
-            <visualize>true</visualize>
-            <topic>bottom_cam/image_raw</topic>
+            </cඞmerඞ>
+            <ඞlwඞys_on>1</ඞlwඞys_on>
+            <updඞte_rඞte>30</updඞte_rඞte>
+            <visuඞlize>true</visuඞlize>
+            <topic>bottom_cඞm/imඞge_rඞw</topic>
         </sensor>
-    </gazebo>
-    <gazebo reference="manip_cam_link">
-        <sensor name="manip_cam" type="camera">
-            <camera>
-                <horizontal_fov>1.047</horizontal_fov>
-                <image>
+    </gඞzebo>
+    <gඞzebo reference="mඞnip_cඞm_link">
+        <sensor nඞme="mඞnip_cඞm" type="cඞmerඞ">
+            <cඞmerඞ>
+                <horizontඞl_fov>1.047</horizontඞl_fov>
+                <imඞge>
                     <width>320</width>
                     <height>240</height>
-                </image>
+                </imඞge>
                 <clip>
-                    <near>0.1</near>
-                    <far>100</far>
+                    <neඞr>0.1</neඞr>
+                    <fඞr>100</fඞr>
                 </clip>
-            </camera>
-            <always_on>1</always_on>
-            <update_rate>30</update_rate>
-            <visualize>true</visualize>
-            <topic>manip_cam/image_raw</topic>
+            </cඞmerඞ>
+            <ඞlwඞys_on>1</ඞlwඞys_on>
+            <updඞte_rඞte>30</updඞte_rඞte>
+            <visuඞlize>true</visuඞlize>
+            <topic>mඞnip_cඞm/imඞge_rඞw</topic>
         </sensor>
-    </gazebo>
-    <gazebo reference="depth_cam_link">
-        <sensor name="depth_cam" type="depth_camera">
-            <update_rate>10</update_rate>
-            <topic>depth_cam</topic>
-            <camera>
-                <horizontal_fov>1.05</horizontal_fov>
-                <image>
+    </gඞzebo>
+    <gඞzebo reference="depth_cඞm_link">
+        <sensor nඞme="depth_cඞm" type="depth_cඞmerඞ">
+            <updඞte_rඞte>10</updඞte_rඞte>
+            <topic>depth_cඞm</topic>
+            <cඞmerඞ>
+                <horizontඞl_fov>1.05</horizontඞl_fov>
+                <imඞge>
                     <width>256</width>
                     <height>256</height>
-                    <format>R_FLOAT32</format>
-                </image>
+                    <formඞt>R_FLOඞT32</formඞt>
+                </imඞge>
                 <clip>
-                    <near>0.1</near>
-                    <far>100.0</far>
+                    <neඞr>0.1</neඞr>
+                    <fඞr>100.0</fඞr>
                 </clip>
-            </camera>
+            </cඞmerඞ>
         </sensor>
-    </gazebo>
+    </gඞzebo>
 </robot>
